File: my_vga_board/my_vga_board.kicad_pcb (KiCad board)
At the start: 2 copper layers, 58.9 x 71.1 mm, 30 parts, among them J1 Barrel_Jack, J2 L77HDE15SD1CH4F, J3 I2C_A, J4 I2C_B, U1 Pico, U2 LM7805_TO220

Commit message: R-2R
Parts:
- added H4: MountingHole, MountingHole:MountingHole_4.3mm_M4, F.Cu at (127.7, 113.6)
- added R20: R, Resistor_SMD:R_0603_1608Metric_Pad0.98x0.95mm_HandSolder, F.Cu at (139.3, 99.4)
- added R21: R, Resistor_SMD:R_0603_1608Metric_Pad0.98x0.95mm_HandSolder, F.Cu at (139.3, 101.9)
- added R22: R, Resistor_SMD:R_0603_1608Metric_Pad0.98x0.95mm_HandSolder, F.Cu at (139.3, 104.4)
- added R23: R, Resistor_SMD:R_0603_1608Metric_Pad0.98x0.95mm_HandSolder, F.Cu at (143.6, 79.3)
- added R24: R, Resistor_SMD:R_0603_1608Metric_Pad0.98x0.95mm_HandSolder, F.Cu at (143.6, 81.9)
- added R25: R, Resistor_SMD:R_0603_1608Metric_Pad0.98x0.95mm_HandSolder, F.Cu at (143.6, 84.4)
- added R26: R, Resistor_SMD:R_0603_1608Metric_Pad0.98x0.95mm_HandSolder, F.Cu at (143.6, 86.9)
- added R27: R, Resistor_SMD:R_0603_1608Metric_Pad0.98x0.95mm_HandSolder, F.Cu at (143.6, 89.4)
- added R28: R, Resistor_SMD:R_0603_1608Metric_Pad0.98x0.95mm_HandSolder, F.Cu at (143.6, 91.9)
- added R29: R, Resistor_SMD:R_0603_1608Metric_Pad0.98x0.95mm_HandSolder, F.Cu at (143.6, 94.4)
- added R30: R, Resistor_SMD:R_0603_1608Metric_Pad0.98x0.95mm_HandSolder, F.Cu at (143.6, 96.9)
- added R31: R, Resistor_SMD:R_0603_1608Metric_Pad0.98x0.95mm_HandSolder, F.Cu at (143.6, 99.4)
- added R32: R, Resistor_SMD:R_0603_1608Metric_Pad0.98x0.95mm_HandSolder, F.Cu at (143.6, 101.9)
- added R33: R, Resistor_SMD:R_0603_1608Metric_Pad0.98x0.95mm_HandSolder, F.Cu at (143.6, 104.4)
- added R34: R, Resistor_SMD:R_0603_1608Metric_Pad0.98x0.95mm_HandSolder, F.Cu at (148.0, 79.3)
- added R35: R, Resistor_SMD:R_0603_1608Metric_Pad0.98x0.95mm_HandSolder, F.Cu at (148.0, 81.9)
- added R36: R, Resistor_SMD:R_0603_1608Metric_Pad0.98x0.95mm_HandSolder, F.Cu at (148.0, 84.4)
- added R37: R, Resistor_SMD:R_0603_1608Metric_Pad0.98x0.95mm_HandSolder, F.Cu at (148.0, 86.9)
- added R38: R, Resistor_SMD:R_0603_1608Metric_Pad0.98x0.95mm_HandSolder, F.Cu at (148.0, 89.4)
- added R39: R, Resistor_SMD:R_0603_1608Metric_Pad0.98x0.95mm_HandSolder, F.Cu at (148.0, 91.9)
- added R40: R, Resistor_SMD:R_0603_1608Metric_Pad0.98x0.95mm_HandSolder, F.Cu at (148.0, 94.4)
- added R41: R, Resistor_SMD:R_0603_1608Metric_Pad0.98x0.95mm_HandSolder, F.Cu at (148.0, 96.9)
- added R42: R, Resistor_SMD:R_0603_1608Metric_Pad0.98x0.95mm_HandSolder, F.Cu at (148.0, 99.4)
- added R43: R, Resistor_SMD:R_0603_1608Metric_Pad0.98x0.95mm_HandSolder, F.Cu at (148.0, 101.9)
- added R44: R, Resistor_SMD:R_0603_1608Metric_Pad0.98x0.95mm_HandSolder, F.Cu at (148.0, 104.4)
- added R45: R, Resistor_SMD:R_0603_1608Metric_Pad0.98x0.95mm_HandSolder, F.Cu at (152.3, 79.3)
- added R46: R, Resistor_SMD:R_0603_1608Metric_Pad0.98x0.95mm_HandSolder, F.Cu at (152.3, 81.9)
- added R47: R, Resistor_SMD:R_0603_1608Metric_Pad0.98x0.95mm_HandSolder, F.Cu at (152.3, 84.4)
- added R48: R, Resistor_SMD:R_0603_1608Metric_Pad0.98x0.95mm_HandSolder, F.Cu at (152.3, 86.9)
- added R49: R, Resistor_SMD:R_0603_1608Metric_Pad0.98x0.95mm_HandSolder, F.Cu at (152.3, 89.4)
- added R50: R, Resistor_SMD:R_0603_1608Metric_Pad0.98x0.95mm_HandSolder, F.Cu at (152.3, 91.9)
- J2: value L77HDE15SD1CH4F -> I2C_A; footprint RPi_Pico:DSUB-15-L77HDE15SD1CH4F -> Connector_PinHeader_2.54mm:PinHeader_1x02_P2.54mm_Horizontal
- J3: value I2C_A -> I2C_B
- J4: value I2C_B -> L77HDE15SD1CH4F; footprint Connector_PinHeader_2.54mm:PinHeader_1x02_P2.54mm_Horizontal -> RPi_Pico:DSUB-15-L77HDE15SD1CH4F
- R1, R2: value 5k -> 47; footprint Resistor_THT:R_Axial_DIN0207_L6.3mm_D2.5mm_P7.62mm_Horizontal -> Resistor_SMD:R_0603_1608Metric_Pad0.98x0.95mm_HandSolder
- R10, R15, R5: value 499 -> R; footprint Resistor_THT:R_Axial_DIN0207_L6.3mm_D2.5mm_P7.62mm_Horizontal -> Resistor_SMD:R_0603_1608Metric_Pad0.98x0.95mm_HandSolder
- R11, R16, R6: value 1k -> R; footprint Resistor_THT:R_Axial_DIN0207_L6.3mm_D2.5mm_P7.62mm_Horizontal -> Resistor_SMD:R_0603_1608Metric_Pad0.98x0.95mm_HandSolder
- R12, R17, R7: value 2k -> R; footprint Resistor_THT:R_Axial_DIN0207_L6.3mm_D2.5mm_P7.62mm_Horizontal -> Resistor_SMD:R_0603_1608Metric_Pad0.98x0.95mm_HandSolder
- R13, R18, R8: value 4.02k -> R; footprint Resistor_THT:R_Axial_DIN0207_L6.3mm_D2.5mm_P7.62mm_Horizontal -> Resistor_SMD:R_0603_1608Metric_Pad0.98x0.95mm_HandSolder
- R14, R19, R9: value 8.06k -> R; footprint Resistor_THT:R_Axial_DIN0207_L6.3mm_D2.5mm_P7.62mm_Horizontal -> Resistor_SMD:R_0603_1608Metric_Pad0.98x0.95mm_HandSolder
- R3, R4: value 47 -> R; footprint Resistor_THT:R_Axial_DIN0207_L6.3mm_D2.5mm_P7.62mm_Horizontal -> Resistor_SMD:R_0603_1608Metric_Pad0.98x0.95mm_HandSolder
- U1: value Pico -> LM7805_TO220; footprint RPi_Pico:RPi_Pico_SMD_TH -> Package_TO_SOT_THT:TO-220-3_Vertical
- U2: value LM7805_TO220 -> Pico; footprint Package_TO_SOT_THT:TO-220-3_Vertical -> RPi_Pico:RPi_Pico_SMD_TH
- moved H3 59.0 mm to (127.7, 103.5)
- moved H2 57.5 mm to (127.7, 93.3)
- moved U2 54.9 mm to (110.6, 80.6), turned to 0 degrees
- moved U1 52.1 mm to (101.8, 111.6)
- moved J4 51.3 mm to (139.1, 60.6)
- moved H1 48.0 mm to (127.7, 83.2)
- moved R4 46.5 mm to (134.9, 86.9), turned to 0 degrees
- moved R3 46.1 mm to (134.9, 84.4), turned to 0 degrees
- moved J1 40.0 mm to (147.3, 111.1), turned to 0 degrees
- moved R2 34.2 mm to (134.9, 81.9), turned to 0 degrees
- moved R9 33.6 mm to (134.9, 99.4)
- moved J3 33.1 mm to (152.1, 115.2)
- moved R1 32.4 mm to (134.9, 79.3), turned to 0 degrees
- moved R15 30.5 mm to (139.3, 86.9)
- moved R8 28.2 mm to (134.9, 96.9)
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Connections:
- C1 pad 1: Net-(C1-Pad1) -> Net-(U1-VI)
- J1 pad 1: Net-(C1-Pad1) -> Net-(U1-VI)
- J2 pad 1: /VGA_R -> /SCL
- J2 pad 2: /VGA_G -> /SDA
- J4 pad 1: /SCL -> /VGA_R
- J4 pad 2: /SDA -> /VGA_G
- R1 pad 1: +3.3V -> /VSYNC
- R1 pad 2: /SCL -> Net-(U2-GPIO17)
- R10 pad 1: /VGA_G -> Net-(R10-Pad1)
- R10 pad 2: /GPIO10 -> GND
- R11 pad 1: /VGA_G -> Net-(R11-Pad1)
- R11 pad 2: /GPIO9 -> Net-(R11-Pad2)
- R12 pad 1: /VGA_G -> Net-(R12-Pad1)
- R12 pad 2: /GPIO8 -> Net-(R12-Pad2)
- R13 pad 1: /VGA_G -> /GPIO1
- R13 pad 2: /GPIO7 -> Net-(R13-Pad2)
- R14 pad 1: /VGA_G -> Net-(R13-Pad2)
- R14 pad 2: /GPIO6 -> Net-(R11-Pad2)
- R15 pad 1: /VGA_B -> /GPIO6
- R15 pad 2: /GPIO15 -> Net-(R15-Pad2)
- R16 pad 1: /VGA_B -> Net-(R15-Pad2)
- R16 pad 2: /GPIO14 -> Net-(R12-Pad2)
- R17 pad 1: /VGA_B -> Net-(R11-Pad2)
- R17 pad 2: /GPIO13 -> Net-(R17-Pad2)
- R18 pad 1: /VGA_B -> Net-(R12-Pad2)
- R18 pad 2: /GPIO12 -> Net-(R18-Pad2)
- R19 pad 1: /VGA_B -> /GPIO2
- R19 pad 2: /GPIO11 -> Net-(R19-Pad2)
- R2 pad 1: +3.3V -> /HSYNC
- R2 pad 2: /SDA -> Net-(U2-GPIO16)
- R3 pad 1: /VSYNC -> /GPIO0
- R3 pad 2: /GPIO17 -> Net-(R3-Pad2)
- R4 pad 1: /HSYNC -> Net-(R3-Pad2)
- R4 pad 2: /GPIO16 -> Net-(R11-Pad1)
- R5 pad 1: /VGA_R -> Net-(R11-Pad1)
- R5 pad 2: /GPIO4 -> Net-(R5-Pad2)
- R6 pad 1: /VGA_R -> Net-(R5-Pad2)
- R6 pad 2: /GPIO3 -> GND
- R7 pad 1: /VGA_R -> /GPIO5
- R7 pad 2: /GPIO2 -> Net-(R7-Pad2)
- R8 pad 1: /VGA_R -> Net-(R7-Pad2)
- R8 pad 2: /GPIO1 -> Net-(R12-Pad1)
- R9 pad 1: /VGA_R -> Net-(R12-Pad1)
- R9 pad 2: /GPIO0 -> Net-(R10-Pad1)
- U1 pad 1: /GPIO0 -> Net-(U1-VI)
- U1 pad 2: /GPIO1 -> GND
- U1 pad 3: GND -> +5V
- U2 pad 1: Net-(C1-Pad1) -> /GPIO0
- U2 pad 2: GND -> /GPIO1
- U2 pad 3: +5V -> GND
Routing:
- net /VGA_R: track 78.7 -> 0.00 mm
- net /VGA_G: track 59.5 -> 0.00 mm
- net /VGA_B: track 41.9 -> 0.00 mm
- net /VSYNC: track 39.6 -> 0.00 mm
- net /HSYNC: track 29.7 -> 0.00 mm
- net /SDA: track 29.3 -> 0.00 mm
- net /SCL: track 29.0 -> 0.00 mm
- net +3.3V: track 22.9 -> 0.00 mm
- net +5V: track 12.2 -> 0.00 mm
- net Net-(C1-Pad1): track 10.9 -> 0.00 mm
- net /GPIO17: track 5.69 -> 0.00 mm
- net /GPIO16: track 5.69 -> 0.00 mm
- net /GPIO9: track 5.40 -> 0.00 mm
- net /GPIO13: track 5.40 -> 0.00 mm
- net /GPIO10: track 5.40 -> 0.00 mm
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- removed copper zone on F.Cu, net GND
Other:
- board outline removed
- board text removed: "SCL"
- board text removed: "Simplified Pico VGA v1 by bunnysamurai"

Commit message: some sound
Parts:
- added D1: LED, LED_THT:LED_D5.0mm, F.Cu at (146.9, 37.3)
- added J5: AudioJack2_Ground, Connector_Audio:Jack_3.5mm_CUI_SJ1-3533NG_Horizontal, F.Cu at (167.2, 104.3)
- added JP1: Open, Jumper:SolderJumper-2_P1.3mm_Open_Pad1.0x1.5mm, F.Cu at (175.2, 99.8)
- added R51: 470, Resistor_SMD:R_0603_1608Metric_Pad0.98x0.95mm_HandSolder, F.Cu at (154.1, 34.8)
- added R52: 470, Resistor_SMD:R_0603_1608Metric_Pad0.98x0.95mm_HandSolder, F.Cu at (154.1, 37.3)
- added R53: 330, Resistor_SMD:R_0603_1608Metric_Pad0.98x0.95mm_HandSolder, F.Cu at (154.1, 39.8)
- added U3: PCM5101A, Package_SO:TSSOP-20_4.4x6.5mm_P0.65mm, F.Cu at (193.1, 123.9)
- added U4: LD3985M33R_SOT23, Package_TO_SOT_SMD:SOT-23-5, F.Cu at (209.3, 74.8)
- U1: footprint Package_TO_SOT_THT:TO-220-3_Vertical -> Package_TO_SOT_THT:TO-220-3_Horizontal_TabDown
- moved J1 127.1 mm to (51.4, 27.6)
- moved J2 127.1 mm to (56.2, 24.6)
- moved J3 127.1 mm to (56.2, 31.8)
- moved U1 86.6 mm to (179.5, 73.4)
- moved R11 80.3 mm to (59.4, 77.1)
- moved R14 78.5 mm to (61.3, 75.1)
- moved R13 78.4 mm to (61.3, 73.6), turned to 180 degrees
- moved R4 78.0 mm to (57.8, 75.1)
- moved R20 78.0 mm to (65.2, 75.1)
- moved R3 77.9 mm to (57.8, 73.6), turned to 180 degrees
- moved R19 77.6 mm to (65.3, 73.6), turned to 180 degrees
- moved R17 77.5 mm to (63.2, 77.1)
- moved R5 76.7 mm to (58.9, 79.1)
- moved R23 76.4 mm to (67.2, 77.1)
- moved R32 76.1 mm to (72.4, 75.1), turned to 180 degrees
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Connections:
- net Net-(U1-VI) renamed VIN
- J4 pad 13: /HSYNC -> Net-(J4-Pad13)
- J4 pad 14: /VSYNC -> Net-(J4-Pad14)
- R1 pad 1: /VSYNC -> /HSYNC
- R1 pad 2: Net-(U2-GPIO17) -> Net-(J4-Pad13)
- R15 pad 1: /GPIO6 -> /GPIO7
- R2 pad 1: /HSYNC -> /VSYNC
- R2 pad 2: Net-(U2-GPIO16) -> Net-(J4-Pad14)
- R21 pad 1: /GPIO7 -> /GPIO8
- R27 pad 1: /GPIO8 -> /GPIO9
- R33 pad 1: /GPIO9 -> /GPIO10
- R35 pad 1: /GPIO10 -> /GPIO11
- R40 pad 1: /GPIO11 -> /GPIO12
- R43 pad 1: /GPIO12 -> /GPIO13
- R46 pad 1: /GPIO13 -> /GPIO14
- R49 pad 1: /GPIO14 -> /GPIO15
- R7 pad 1: /GPIO5 -> /GPIO6
- U2 pad 21: Net-(U2-GPIO16) -> /HSYNC
- U2 pad 22: Net-(U2-GPIO17) -> /VSYNC
- U2 pad 31: unconnected-(U2-GPIO26_ADC0-Pad31) -> /GPIO26
- U2 pad 32: unconnected-(U2-GPIO27_ADC1-Pad32)_0 -> /GPIO27
- U2 pad 34: unconnected-(U2-GPIO28_ADC2-Pad34) -> /GPIO28
- U2 pad 36: +3.3V -> +3V3 (OUT)
- U2 pad 40: unconnected-(U2-VBUS-Pad40)_0 -> Net-(JP1-A)
Routing:
- net Net-(R42-Pad2): track 0.00 -> 4.96 mm
- net Net-(R39-Pad2): track 0.00 -> 4.83 mm
- net /GPIO6: track 0.00 -> 4.76 mm
- net /GPIO8: track 0.00 -> 4.71 mm
- net /GPIO11: track 0.00 -> 4.60 mm
- net /HSYNC: track 0.00 -> 4.54 mm
- net Net-(R12-Pad1): track 0.00 -> 4.54 mm
- net /GPIO1: track 0.00 -> 4.53 mm
- net /VSYNC: track 0.00 -> 4.51 mm
- net /GPIO3: track 0.00 -> 4.48 mm
- net /GPIO7: track 0.00 -> 4.42 mm
- net /GPIO9: track 0.00 -> 4.35 mm
- net Net-(R11-Pad1): track 0.00 -> 4.30 mm
- net /GPIO10: track 0.00 -> 4.29 mm
- net Net-(R17-Pad2): track 0.00 -> 4.25 mm
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- removed copper zone on B.Cu, net GND
